File: esp8266/leaky/pcb/leaky/leaky.sch (KiCad schematic (older format))
At the start: 31 parts, among them J1 UART, J2 extra pins, Q1 BC327, SW1 sensing loop, U1 DD0405MA, U2 ESP-12F

Commit message: leaky: Adjust RX TX
Other:
- note added: "VBUS voltage has to be 3V3, not 5V!\nIf you provide power through VBUS, remove batteries first.\n\nTo flash program: \n 1. Short jumper PROG\n 2. Connect UART (RXD->TX, TXD->RX)\n 3. Short jumper TURN_ON\n"
- note removed: "VBUS voltage has to be 3V3, not 5V!\nIf you provide power through VBUS, remove batteries first.\nTo flash program: \n 1. Short jumper PROG\n 2. Connect UART\n 3. Short jumper TURN_ON\n"
Changed lines of the file:
@@
 Mounting holes
 Text Notes 4770 4450 0    50   ~ 0
-VBUS voltage has to be 3V3, not 5V!\nIf you provide power through VBUS, remove batteries first.\nTo flash program: \n  1. Short jumper PROG\n  2. Connect UART\n  3. Short jumper TURN_ON\n
+VBUS voltage has to be 3V3, not 5V!\nIf you provide power through VBUS, remove batteries first.\n\nTo flash program: \n  1. Short jumper PROG\n  2. Connect UART (RXD->TX, TXD->RX)\n  3. Short jumper TURN_ON\n
 Wire Wire Line
 	1510 3190 1380 3190

Commit message: leaky: Send v1.0 to jlcpcb
Other:
- note added: "Current consumption in standby mode is about 30-40 uA"
Changed lines of the file:
@@
 Wire Wire Line
 	2950 1000 3200 1000
+Text Notes 1810 1860 0    50   ~ 0
+Current consumption in standby mode is about 30-40 uA
 $EndSCHEMATC
