File: nrf52840/MS88SF2_breakout/MS88SF2_breakout_panel.kicad_pcb (KiCad board)
At the start: 2 copper layers, 100 x 100 mm, 198 parts, among them J1 Conn_01x14_Male, J2 Conn_01x14_Male, U1 MS88SF2

Commit message: nrf5: Send to a fab
Other:
- board text added: "JLCJLCJLCJLC"
