File: esp32/ledstrip/!pcb/!pcb.kicad_pcb (KiCad board)
At the start: 2 copper layers, 44 x 77 mm, 18 parts, among them J1 Barrel_Jack_Switch, J2 Conn_01x03, SW1 SW_SPST, U1 ESP32 MINI, U2 INMP441

Commit message: ledstrip: Add logo
Parts:
- added G***: LOGO, _my:logo, F.Cu at (52.2, 63.0)

Commit message: ledstrip: Send to a fab
Other:
- rule trace_min: 0.2 -> 0.25
- board text added: "INMP441"
- board text added: "MINI D1 ESP32"
- board text added: "WS2812B"
- board text added: "revA"
- board text removed: "v1.0"
